Commit message: added gazebo_grasp_plugin functionality to both oberon manipulators

File: rexrov_dual_oberon/rexrov_dual_oberon_description/robots/rexrov_dual_oberon7.xacro (robot description, xacro)
@@ -45,8 +45,35 @@
   </xacro:oberon7>
   <gazebo>
-      <plugin name="gazebo_ros_control" filename="libgazebo_ros_control.so">
-        <robotNamespace>/$(arg namespace)</robotNamespace>
-        <robotParam>/$(arg namespace)/robot_description</robotParam>
-      </plugin>
+    <plugin name="gazebo_ros_control" filename="libgazebo_ros_control.so">
+      <robotNamespace>/$(arg namespace)</robotNamespace>
+      <robotParam>/$(arg namespace)/robot_description</robotParam>
+    </plugin>
+    <plugin name="gazebo_grasp_fix" filename="libgazebo_grasp_fix.so">
+      <arm>
+        <arm_name>oberon_L</arm_name>
+        <palm_link> oberon_L/end_effector </palm_link>
+        <gripper_link> oberon_L/finger_left </gripper_link>
+        <gripper_link> oberon_L/finger_right </gripper_link>
+        <gripper_link> oberon_L/finger_tip_left </gripper_link>
+        <gripper_link> oberon_L/finger_tip_right </gripper_link>
+        <!-- <gripper_link> ... </gripper_link> -->
+      </arm>
+      <arm>
+        <arm_name>oberon_R</arm_name>
+        <palm_link> oberon_R/end_effector </palm_link>
+        <gripper_link> oberon_R/finger_left </gripper_link>
+        <gripper_link> oberon_R/finger_right </gripper_link>
+        <gripper_link> oberon_R/finger_tip_left </gripper_link>
+        <gripper_link> oberon_R/finger_tip_right </gripper_link>
+        <!-- <gripper_link> ... </gripper_link> -->
+      </arm>
+      <forces_angle_tolerance>100</forces_angle_tolerance>
+      <update_rate>4</update_rate>
+      <grip_count_threshold>4</grip_count_threshold>
+      <max_grip_count>8</max_grip_count>
+      <release_tolerance>0.005</release_tolerance>
+      <disable_collisions_on_attach>false</disable_collisions_on_attach>
+      <contact_topic>__default_topic__</contact_topic>
+    </plugin>
   </gazebo>
   <!-- Joint state publisher plugin -->

File: uuv_manipulators-master/oberon7/oberon7_description/urdf/parallel_gripper.xacro (robot description, xacro)
@@ -70,5 +70,5 @@
         <origin xyz="0.0444267 0.0391376 0" rpy="0 0 0"/>
         <axis xyz="0 0 1"/>
-        <dynamics damping="5" friction="10"/>
+        <dynamics damping="5" friction="1"/>
         <!-- <dynamics damping="5" friction="0"/> -->
         <limit effort="${gripper_effort}" lower="0" upper="${PI*0.3333}" velocity="${gripper_velocity}"/>
@@ -101,5 +101,5 @@
         <origin xyz="0.06431 0 0" rpy="${PI} 0 0"/>
         <axis xyz="0 0 1"/>
-        <dynamics damping="5" friction="10"/>
+        <dynamics damping="5" friction="1"/>
         <!-- <dynamics damping="5" friction="0"/> -->
         <limit effort="0" lower="0" upper="0" velocity="0"/>
@@ -131,5 +131,5 @@
         <origin xyz="0.0444267 -0.0391376 0" rpy="${PI} ${PI} ${PI}"/>
         <axis xyz="0 0 -1"/>
-        <dynamics damping="5" friction="10"/>
+        <dynamics damping="5" friction="1"/>
         <!-- <dynamics damping="10" friction="0"/> -->
         <limit effort="${gripper_effort}" lower="0" upper="${PI*0.3333}" velocity="${gripper_velocity}"/>
@@ -162,5 +162,5 @@
         <origin xyz="0.06431 0 0" rpy="0 0 0"/>
         <axis xyz="0 0 1"/>
-        <dynamics damping="5" friction="10"/>
+        <dynamics damping="5" friction="1"/>
         <!-- <dynamics damping="5" friction="0"/> -->
         <limit effort="0" lower="0" upper="0" velocity="0"/>
