Commit message: Created lite rexrov model

File: rexrov_dual_oberon/rexrov_dual_oberon_description/objects/perch_structure/perch_structure.urdf (robot description, URDF)
Before this commit: robot perch_structure, 14 links, 13 joints
Links:
- added link sup1, mass 1.0; collision cylinder length=1 radius=0.02; visual cylinder length=1 radius=0.02
- added link sup2, mass 1.0; collision cylinder length=1 radius=0.02; visual cylinder length=1 radius=0.02
- added link sup3, mass 1.0; collision cylinder length=1 radius=0.02; visual cylinder length=1 radius=0.02
- added link sup4, mass 1.0; collision cylinder length=1 radius=0.02; visual cylinder length=1 radius=0.02
- added link sup5, mass 1.0; collision cylinder length=1 radius=0.02; visual cylinder length=1 radius=0.02
- added link sup6, mass 1.0; collision cylinder length=1 radius=0.02; visual cylinder length=1 radius=0.02
- added link sup7, mass 1.0; collision cylinder length=1 radius=0.02; visual cylinder length=1 radius=0.02
- added link sup8, mass 1.0; collision cylinder length=1 radius=0.02; visual cylinder length=1 radius=0.02
- link base_1: mass 50.0 -> 5.0
- link base_2: mass 50.0 -> 5.0
- link base_3: mass 50.0 -> 5.0
- link base_4: mass 50.0 -> 5.0
- link base_5: mass 50.0 -> 5.0
Joints:
- added joint sup_fix1: type fixed, parent pillar1, child sup1, origin xyz=1 0 0.5
- added joint sup_fix2: type fixed, parent pillar1, child sup2, origin xyz=2 0 0.5
- added joint sup_fix3: type fixed, parent pillar1, child sup3, origin xyz=0 1 0.5
- added joint sup_fix4: type fixed, parent pillar1, child sup4, origin xyz=0 2 0.5
- added joint sup_fix5: type fixed, parent pillar1, child sup5, origin xyz=-1 0 0.5
- added joint sup_fix6: type fixed, parent pillar1, child sup6, origin xyz=-2 0 0.5
- added joint sup_fix7: type fixed, parent pillar1, child sup7, origin xyz=0 -1 0.5
- added joint sup_fix8: type fixed, parent pillar1, child sup8, origin xyz=0 -2 0.5
