Commit message: added smooth 5th order polynomial manipulator joint publisher

File: rexrov_dual_oberon/oberon7_lite/urdf/serial_arm_lite_backup.xacro (robot description, xacro)
@@ -47,5 +47,5 @@
                 <origin xyz="0 0 0" rpy="0 0 0"/>
                 <geometry>
-                    <cylinder radius="1e-9" length="1e-9" />
+                    <mesh filename="file://$(find oberon7_lite)/meshes/serial_arm/collision/Base.stl"/>
                 </geometry>
             </collision>
@@ -68,5 +68,5 @@
                 <origin xyz="${shoulder_link_com}" rpy="0 0 0"/>
                 <geometry>
-                    <cylinder radius="1e-9" length="1e-9" />
+                    <cylinder radius="${0.5 * shoulder_link_width}" length="${shoulder_link_height}" />
                 </geometry>
             </collision>
@@ -79,5 +79,5 @@
             <!-- <dynamics damping="1" friction="150"/> -->
             <dynamics damping="1" friction="0.50"/>
-            <limit lower="${-180 * d2r}" upper="${180 * d2r}" velocity="0.17" effort="200"/>
+            <limit lower="${-60 * d2r}" upper="${60 * d2r}" velocity="0.17" effort="200"/>
             <!-- <limit lower="${-60 * d2r}" upper="${60 * d2r}" velocity="0.17" effort="1000"/> -->
         </joint>
@@ -100,5 +100,5 @@
                 <origin xyz="${upper_arm_com}" rpy="0 ${0.5*pi} 0"/>
                 <geometry>
-                    <cylinder radius="1e-9" length="1e-9" />
+                    <cylinder radius="${0.5 * upper_arm_width}" length="${upper_arm_length}"/>
                 </geometry>
             </collision>
@@ -133,5 +133,5 @@
                 <origin xyz="${elbow_link_com}" rpy="0 ${0.5*pi} ${0.5*pi}"/>
                 <geometry>
-                    <cylinder radius="1e-9" length="1e-9" />
+                    <cylinder radius="${0.5 * elbow_link_height}" length="${elbow_link_length}"/>
                 </geometry>
             </collision>
@@ -166,5 +166,5 @@
                 <origin xyz="${forearm_com}" rpy="0 0 0"/>
                 <geometry>
-                    <cylinder radius="1e-9" length="1e-9" />
+                    <cylinder radius="${0.5 * forearm_width}" length="${forearm_height}"/>
                 </geometry>
             </collision>
@@ -200,5 +200,5 @@
                 <origin xyz="${wrist_com}" rpy="0 ${0.5*pi} 0"/>
                 <geometry>
-                    <cylinder radius="1e-9" length="1e-9" />
+                    <cylinder radius="${0.5 * wrist_height}" length="${wrist_length}"/>
                 </geometry>
             </collision>

File: rexrov_triple_oberon/rexrov_triple_oberon_description/robots/rexrov_triple.xacro (robot description, xacro)
@@ -5,7 +5,7 @@
   <xacro:arg name="inertial_reference_frame" default="world"/>
   <!-- Include the ROV macro file -->
-  <xacro:include filename="$(find uuv_descriptions)/urdf/rexrov_base.xacro"/>
-  <xacro:include filename="$(find uuv_descriptions)/urdf/rexrov.gazebo.xacro"/>
-  <xacro:include filename="$(find oberon7_description)/robots/oberon7_default.xacro" />
+  <xacro:include filename="$(find rexrov_triple_oberon_description)/urdf/rexrov_lite_base.xacro"/>
+  <xacro:include filename="$(find rexrov_triple_oberon_description)/urdf/rexrov_lite.gazebo.xacro"/>
+  <xacro:include filename="$(find oberon7_lite)/robots/oberon7_lite.xacro" />
   <!-- Create the ROV -->
   <xacro:rexrov_base
@@ -26,9 +26,12 @@
     </gazebo>
   </xacro:rexrov_base>
-  <xacro:oberon7 namespace="oberon_L" parent="$(arg namespace)/base_link">
+  <xacro:oberon7 namespace="oberon1" parent="$(arg namespace)/base_link">
     <origin xyz="1.3 0.5 -0.615" rpy="0 0 0"/>
   </xacro:oberon7>
-  <xacro:oberon7 namespace="oberon_R" parent="$(arg namespace)/base_link">
+  <xacro:oberon7 namespace="oberon2" parent="$(arg namespace)/base_link">
     <origin xyz="1.3 -0.5 -0.615" rpy="0 0 0"/>
+  </xacro:oberon7>
+  <xacro:oberon7 namespace="oberon3" parent="$(arg namespace)/base_link">
+    <origin xyz="1.3 0.0 0.3" rpy="0 0 0"/>
   </xacro:oberon7>
   <gazebo>
@@ -39,26 +42,36 @@
     <plugin name="gazebo_grasp_fix" filename="libgazebo_grasp_fix.so">
       <arm>
-        <arm_name>oberon_L</arm_name>
-        <palm_link> oberon_L/end_effector </palm_link>
-        <gripper_link> oberon_L/finger_left </gripper_link>
-        <gripper_link> oberon_L/finger_right </gripper_link>
-        <gripper_link> oberon_L/finger_tip_left </gripper_link>
-        <gripper_link> oberon_L/finger_tip_right </gripper_link>
+        <arm_name>oberon1</arm_name>
+        <palm_link> oberon1/end_effector </palm_link>
+        <gripper_link> oberon1/finger_left </gripper_link>
+        <gripper_link> oberon1/finger_right </gripper_link>
+        <gripper_link> oberon1/finger_tip_left </gripper_link>
+        <gripper_link> oberon1/finger_tip_right </gripper_link>
         <!-- <gripper_link> ... </gripper_link> -->
       </arm>
       <arm>
-        <arm_name>oberon_R</arm_name>
-        <palm_link> oberon_R/end_effector </palm_link>
-        <gripper_link> oberon_R/finger_left </gripper_link>
-        <gripper_link> oberon_R/finger_right </gripper_link>
-        <gripper_link> oberon_R/finger_tip_left </gripper_link>
-        <gripper_link> oberon_R/finger_tip_right </gripper_link>
+        <arm_name>oberon2</arm_name>
+        <palm_link> oberon2/end_effector </palm_link>
+        <gripper_link> oberon2/finger_left </gripper_link>
+        <gripper_link> oberon2/finger_right </gripper_link>
+        <gripper_link> oberon2/finger_tip_left </gripper_link>
+        <gripper_link> oberon2/finger_tip_right </gripper_link>
         <!-- <gripper_link> ... </gripper_link> -->
       </arm>
-      <forces_angle_tolerance>100</forces_angle_tolerance>
+      <arm>
+        <arm_name>oberon3</arm_name>
+        <palm_link> oberon3/end_effector </palm_link>
+        <gripper_link> oberon3/finger_left </gripper_link>
+        <gripper_link> oberon3/finger_right </gripper_link>
+        <gripper_link> oberon3/finger_tip_left </gripper_link>
+        <gripper_link> oberon3/finger_tip_right </gripper_link>
+        <!-- <gripper_link> ... </gripper_link> -->
+      </arm>
+      <forces_angle_tolerance>90</forces_angle_tolerance>
       <update_rate>4</update_rate>
       <grip_count_threshold>4</grip_count_threshold>
       <max_grip_count>8</max_grip_count>
       <release_tolerance>0.005</release_tolerance>
+      <!-- <release_tolerance>0.005</release_tolerance> -->
       <disable_collisions_on_attach>false</disable_collisions_on_attach>
       <contact_topic>__default_topic__</contact_topic>
